File: STM32_LQFP64/STM32_LQFP64/STM32_FOC_Board.kicad_pcb (KiCad board)
At the start: 4 copper layers, 22 x 26.1 mm, 46 parts, among them J1 Bus_M.2_Socket_E, SW1 TS342A2P-WZ, SW2 TS342A2P-WZ, U1 STM32F446RETx, U2 ME6217C33M5G, X1 FC-12M32.768KHZ7PF20PPM, X2 7R24000E12UBE

Commit message: "UPDATE LQFP32 AND LQFP64"
Changed lines of the file:
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@@
   (gr_line (start 129 81.83) (end 138.4808 81.83) (layer "Edge.Cuts") (width 0.05))
   (gr_line (start 141.478 81.8388) (end 151 81.8388) (layer "Edge.Cuts") (width 0.05))
-  (gr_arc (start 141.478 81.8388) (mid 139.974988 83.336936) (end 138.4808 81.83) (layer "Edge.Cuts") (width 0.05))
+  (gr_arc (start 141.478 81.8388) (mid 139.974988 83.336937) (end 138.4808 81.83) (layer "Edge.Cuts") (width 0.05))
   (gr_line (start 129 107.8875) (end 129 81.83) (layer "Edge.Cuts") (width 0.05))
   (gr_line (start 143.23 111.88) (end 149.93 111.88) (layer "Margin") (width 0.15))
